File: larsskj-001.kicad_pcb (KiCad board)
At the start: 2 copper layers, 73.7 x 41.9 mm, 11 parts, among them J1 In, J2 TLC in, J3 VCC, J4 TLC out, J5 Out

Commit message: README.md modified
Parts:
- removed REF**: OSHW-Logo_5.7x6mm_SilkScreen, Symbol:OSHW-Logo_5.7x6mm_SilkScreen
- removed REF** (x4): MountingHole_3.2mm_M3, MountingHole:MountingHole_3.2mm_M3
- J3: value VCC -> 1888687; footprint TerminalBlock:TerminalBlock_bornier-2_P5.08mm -> 1888687:SHDR2W90P0X508_1X2_1016X950X1500P
